Commit message: 模型改為實機重量 (本體 875 g + LiDAR 45 g)、LiDAR 後移、RL v6
- 質量: 官方 URDF 各連桿等比例放大到本體 875 g, DOGZILLA S2 LiDAR 45 g
- LiDAR 位置: Gazebo 掃描 8 個前後位置, 由官方 x=-0.0167 後移到 x=-0.06
  (質心較接近四腳支撐中心, 官方位置之前會翻倒), 自身回波過濾範圍跟著調整
- 關節 PID p 8 -> 14 (新重量下 p<=12 撐不住, p>=17 顫振)
- RL v6: 依 920 g 模型的 Gazebo 實測速度反應, 以 v5 權重為起點接續訓練 2M 步;
  project3 場地 Gazebo benchmark 7/7 到達、0 碰撞、未翻倒 (單次執行)
- 速度上限維持 0.15 m/s (0.20 m/s 急起急停會翻倒, tools/startstop_test.py)
- 新工具: tune_sweep.sh, com_check.py, startstop_test.py, stand_drift.py;
  train.py 增加 --init (接續訓練)
- 文件與結果紀錄更新 (README, SETUP, results/)

Co-Authored-By: Claude Opus 5.5 <noreply@anthropic.com>

File: sim_env/description/dogzilla_s1_official.urdf.xacro (robot description, xacro)
@@ -9,6 +9,6 @@
     <inertial>
       <origin xyz="0.00520835146477011 -0.000260539720599709 0.0280591836024867" rpy="0 0 0" />
-      <mass value="0.387351847505872" />
-      <inertia ixx="0.000190614924105559" ixy="1.611909782579E-06" ixz="-3.19577698047172E-06" iyy="0.0010563840813291" iyz="-1.54888786284979E-06" izz="0.00118548753067654" />
+      <mass value="0.555142" />
+      <inertia ixx="0.000273184" ixy="2.31015e-06" ixz="-4.5801e-06" iyy="0.00151398" iyz="-2.21982e-06" izz="0.00169901" />
     </inertial>
     <visual>
@@ -25,6 +25,6 @@
     <inertial>
       <origin xyz="-0.0139720018610026 0.0250894092965121 0.00927328896542384" rpy="0 0 0" />
-      <mass value="0.019600254805245" />
-      <inertia ixx="5.89203493378017E-06" ixy="-5.67038080686865E-07" ixz="-2.62883769311083E-07" iyy="3.7904205321723E-06" iyz="-1.16491568847576E-06" izz="6.88837034802653E-06" />
+      <mass value="0.0280906" />
+      <inertia ixx="8.44431e-06" ixy="-8.12664e-07" ixz="-3.76758e-07" iyy="5.43233e-06" iyz="-1.66953e-06" izz="9.87223e-06" />
     </inertial>
     <visual>
@@ -48,6 +48,6 @@
     <inertial>
       <origin xyz="-0.00689428079248722 -0.0186700000000002 -0.0299480398915498" rpy="0 0 0" />
-      <mass value="0.012342949675616" />
-      <inertia ixx="5.47497407669945E-06" ixy="-3.81090641763637E-22" ixz="5.64425515319236E-21" iyy="4.86023562858699E-06" iyz="1.43987804089399E-12" izz="1.83454593627849E-06" />
+      <mass value="0.0176896" />
+      <inertia ixx="7.84659e-06" ixy="-5.46169e-22" ixz="8.08919e-21" iyy="6.96556e-06" iyz="2.06359e-12" izz="2.62922e-06" />
     </inertial>
     <visual>
@@ -71,6 +71,6 @@
     <inertial>
       <origin xyz="-0.0167811557825132 -0.0183250059303989 -0.03162385840477" rpy="0 0 0" />
-      <mass value="0.022687879462132" />
-      <inertia ixx="1.41147289858082E-05" ixy="-5.34206016944144E-13" ixz="-9.81905906721924E-07" iyy="1.36483004430885E-05" iyz="-2.32220795182774E-12" izz="1.39274465973039E-06" />
+      <mass value="0.0325157" />
+      <inertia ixx="2.02289e-05" ixy="-7.6561e-13" ixz="-1.40724e-06" iyy="1.95604e-05" iyz="-3.32813e-12" izz="1.99604e-06" />
     </inertial>
     <visual>
@@ -94,6 +94,6 @@
     <inertial>
       <origin xyz="-0.0139720018610026 -0.0250894092965121 0.00927328896542384" rpy="0 0 0" />
-      <mass value="0.019600254805245" />
-      <inertia ixx="5.89203493378017E-06" ixy="5.67038080686865e-07" ixz="-2.62883769311083E-07" iyy="3.7904205321723E-06" iyz="1.16491568847576e-06" izz="6.88837034802653E-06" />
+      <mass value="0.0280906" />
+      <inertia ixx="8.44431e-06" ixy="8.12664e-07" ixz="-3.76758e-07" iyy="5.43233e-06" iyz="1.66953e-06" izz="9.87223e-06" />
     </inertial>
     <visual>
@@ -117,6 +117,6 @@
     <inertial>
       <origin xyz="-0.00689428079248688 0.018700000000002 -0.0299480398915499" rpy="0 0 0" />
-      <mass value="0.0123429496756159" />
-      <inertia ixx="5.47497407669944E-06" ixy="-2.0611276716309E-20" ixz="1.96257242900458E-21" iyy="4.86023562858698E-06" iyz="1.43987803985982E-12" izz="1.83454593627847E-06" />
+      <mass value="0.0176896" />
+      <inertia ixx="7.84659e-06" ixy="-2.95395e-20" ixz="2.81271e-21" iyy="6.96556e-06" iyz="2.06359e-12" izz="2.62922e-06" />
     </inertial>
     <visual>
@@ -140,6 +140,6 @@
     <inertial>
       <origin xyz="-0.016781155771109 0.0183249940632203 -0.0316238583795284" rpy="0 0 0" />
-      <mass value="0.0226878794123114" />
-      <inertia ixx="1.41147289746255E-05" ixy="-5.3440270556883E-13" ixz="-9.81905905136456E-07" iyy="1.3648300431669E-05" iyz="-2.32170698199082E-12" izz="1.39274465829374E-06" />
+      <mass value="0.0325157" />
+      <inertia ixx="2.02289e-05" ixy="-7.65892e-13" ixz="-1.40724e-06" iyy="1.95604e-05" iyz="-3.32741e-12" izz="1.99604e-06" />
     </inertial>
     <visual>
@@ -163,6 +163,6 @@
     <inertial>
       <origin xyz="-0.0139720018610022 0.0250894092965121 0.00927328896542402" rpy="0 0 0" />
-      <mass value="0.019600254805245" />
-      <inertia ixx="5.89203493378016E-06" ixy="-5.67038080686868E-07" ixz="-2.62883769311102E-07" iyy="3.79042053217232E-06" iyz="-1.16491568847579E-06" izz="6.8883703480265E-06" />
+      <mass value="0.0280906" />
+      <inertia ixx="8.44431e-06" ixy="-8.12664e-07" ixz="-3.76758e-07" iyy="5.43233e-06" iyz="-1.66953e-06" izz="9.87223e-06" />
     </inertial>
     <visual>
@@ -186,6 +186,6 @@
     <inertial>
       <origin xyz="-0.00689428079248695 -0.0186700000000005 -0.0299480398915495" rpy="0 0 0" />
-      <mass value="0.0123429496756159" />
-      <inertia ixx="5.47497407669944E-06" ixy="-2.75633243799764E-21" ixz="9.32745289581667E-21" iyy="4.86023562858698E-06" iyz="1.4398780610445E-12" izz="1.83454593627848E-06" />
+      <mass value="0.0176896" />
+      <inertia ixx="7.84659e-06" ixy="-3.9503e-21" ixz="1.33679e-20" iyy="6.96556e-06" iyz="2.06359e-12" izz="2.62922e-06" />
     </inertial>
     <visual>
@@ -209,6 +209,6 @@
     <inertial>
       <origin xyz="-0.0167811557787652 -0.0183250059325003 -0.0316238584061345" rpy="0 0 0" />
-      <mass value="0.0226878794439316" />
-      <inertia ixx="1.41147289784473E-05" ixy="-5.34101678210922E-13" ixz="-9.81905906147013E-07" iyy="1.36483004357316E-05" iyz="-2.32069575705543E-12" izz="1.39274465908676E-06" />
+      <mass value="0.0325157" />
+      <inertia ixx="2.02289e-05" ixy="-7.6546e-13" ixz="-1.40724e-06" iyy="1.95604e-05" iyz="-3.32596e-12" izz="1.99604e-06" />
     </inertial>
     <visual>
@@ -232,6 +232,6 @@
     <inertial>
       <origin xyz="-0.0139720018610026 -0.0250894092965121 0.00927328896542384" rpy="0 0 0" />
-      <mass value="0.019600254805245" />
-      <inertia ixx="5.89203493378017E-06" ixy="5.67038080686865e-07" ixz="-2.62883769311083E-07" iyy="3.7904205321723E-06" iyz="1.16491568847576e-06" izz="6.88837034802653E-06" />
+      <mass value="0.0280906" />
+      <inertia ixx="8.44431e-06" ixy="8.12664e-07" ixz="-3.76758e-07" iyy="5.43233e-06" iyz="1.66953e-06" izz="9.87223e-06" />
     </inertial>
     <visual>
@@ -255,6 +255,6 @@
     <inertial>
       <origin xyz="-0.00689428079248684 0.0187000000000015 -0.0299480398915497" rpy="0 0 0" />
-      <mass value="0.0123429496756159" />
-      <inertia ixx="5.47497407669943E-06" ixy="-1.59437966027726E-21" ixz="2.38691803281188E-22" iyy="4.86023562858697E-06" iyz="1.43987807159176E-12" izz="1.83454593627849E-06" />
+      <mass value="0.0176896" />
+      <inertia ixx="7.84659e-06" ixy="-2.28502e-21" ixz="3.42087e-22" iyy="6.96556e-06" iyz="2.06359e-12" izz="2.62922e-06" />
     </inertial>
     <visual>
@@ -278,6 +278,6 @@
     <inertial>
       <origin xyz="-0.0167811557016845 0.0183249940379433 -0.0316238581313005" rpy="0 0 0" />
-      <mass value="0.0226878792028959" />
-      <inertia ixx="1.41147288978932E-05" ixy="-5.37750477164225E-13" ixz="-9.81905884621754E-07" iyy="1.36483003526844E-05" iyz="-2.33519052107278E-12" izz="1.39274464946125E-06" />
+      <mass value="0.0325157" />
+      <inertia ixx="2.02289e-05" ixy="-7.7069e-13" ixz="-1.40724e-06" iyy="1.95604e-05" iyz="-3.34673e-12" izz="1.99604e-06" />
     </inertial>
     <visual>
@@ -301,6 +301,6 @@
     <inertial>
       <origin xyz="-0.0141667877097374 -4.70243546289578E-05 -0.000117154201057887" rpy="0 0 0" />
-      <mass value="0.00465716120355248" />
-      <inertia ixx="3.06225211138596E-07" ixy="-1.92519366340594E-09" ixz="5.22083640009109E-09" iyy="3.69724180703298E-07" iyz="2.22463439295763E-09" izz="3.81829903495435E-07" />
+      <mass value="0.00667452" />
+      <inertia ixx="4.38874e-07" ixy="-2.75914e-09" ixz="7.48236e-09" iyy="5.29879e-07" iyz="3.18829e-09" izz="5.47228e-07" />
     </inertial>
     <visual>
@@ -323,6 +323,6 @@
     <inertial>
       <origin xyz="3.78566923279477E-05 -0.000119937093508327 -0.022798439512917" rpy="0 0 0" />
-      <mass value="0.0141156733693049" />
-      <inertia ixx="2.42577727195545E-06" ixy="-7.70141087552742E-09" ixz="6.54011918414534E-09" iyy="2.37021015047955E-06" iyz="6.61859556534528E-09" izz="4.25931212063486E-06" />
+      <mass value="0.045" />
+      <inertia ixx="7.73325e-06" ixy="-2.45517e-08" ixz="2.08495e-08" iyy="7.5561e-06" iyz="2.10997e-08" izz="1.35785e-05" />
     </inertial>
     <visual>
@@ -337,5 +337,5 @@
     </link>
   <joint name="laser_Joint" type="fixed">
-    <origin xyz="-0.016732 4.4164E-05 0.10335" rpy="0 0 0" />
+    <origin xyz="-0.06 4.4164E-05 0.10335" rpy="0 0 0" />
     <parent link="base_link" />
     <child link="laser_link" />
